File: KiCad/Mainboard/Arduino_UNO.sch (KiCad schematic (older format))
At the start: 11 parts, among them IC1 ATMEGA328P-P, P24 CONN_3X2, P25 CONN_6, SW2 SW_PUSH, X1 16.00MHz

Commit message: Initial Board Layout
Parts:
- added D8: 1N4001, symbol DIODE
Connections:
- net +5V: now also D8.2 (K)
- net at C5.1, IC1.1 ((PCINT14/~RESET~)PC6), P24.5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: now also D8.1 (A)
Other:
- moved on the sheet: R10
Changed lines of the file:
@@
 $EndDescr
 $Comp
-L GND #PWR035
+L GND #PWR042
 U 1 1 535D55D8
 P 1900 4100
-F 0 "#PWR035" H 1900 4100 30  0001 C CNN
+F 0 "#PWR042" H 1900 4100 30  0001 C CNN
 F 1 "GND" H 1900 4030 30  0001 C CNN
 F 2 "" H 1900 4100 60  0000 C CNN
@@
 $EndComp
 $Comp
-L +5V #PWR036
+L +5V #PWR043
 U 1 1 535D5743
 P 1900 1600
-F 0 "#PWR036" H 1900 1690 20  0001 C CNN
+F 0 "#PWR043" H 1900 1690 20  0001 C CNN
 F 1 "+5V" H 1900 1690 30  0000 C CNN
 F 2 "" H 1900 1600 60  0000 C CNN
@@
 $EndComp
 $Comp
-L +5V #PWR037
+L +5V #PWR044
 U 1 1 535D874F
 P 5800 2400
-F 0 "#PWR037" H 5800 2490 20  0001 C CNN
+F 0 "#PWR044" H 5800 2490 20  0001 C CNN
 F 1 "+5V" H 5800 2490 30  0000 C CNN
 F 2 "" H 5800 2400 60  0000 C CNN
@@
 $EndComp
 $Comp
-L GND #PWR038
+L GND #PWR045
 U 1 1 535D875A
 P 5800 2800
-F 0 "#PWR038" H 5800 2800 30  0001 C CNN
+F 0 "#PWR045" H 5800 2800 30  0001 C CNN
 F 1 "GND" H 5800 2730 30  0001 C CNN
 F 2 "" H 5800 2800 60  0000 C CNN
@@
 FTDI
 $Comp
-L GND #PWR039
+L GND #PWR046
 U 1 1 535D90FA
 P 4900 3700
-F 0 "#PWR039" H 4900 3700 30  0001 C CNN
+F 0 "#PWR046" H 4900 3700 30  0001 C CNN
 F 1 "GND" H 4900 3630 30  0001 C CNN
 F 2 "" H 4900 3700 60  0000 C CNN
@@
 ICSP
 $Comp
-L CRYSTAL X1
-U 1 1 535DA8D4
-P 4850 1200
-F 0 "X1" H 4850 1350 60  0000 C CNN
-F 1 "16.00MHz" H 4850 1050 60  0000 C CNN
-F 2 "" H 4850 1200 60  0000 C CNN
-F 3 "" H 4850 1200 60  0000 C CNN
-	1    4850 1200
-	0    1    1    0
-$EndComp
-$Comp
 L ATMEGA328P-P IC1
 U 1 1 535D55C4
@@
 	1    2950 2800
 	1    0    0    -1
-$EndComp
-$Comp
-L Capacitor-General_EN60617-4_04-02-01_Date20121108 C6
-U 1 1 535DAAC1
-P 5150 900
-F 0 "C6" H 5200 1000 50  0000 L CNN
-F 1 "22pf" H 4950 1000 50  0000 L CNN
-F 2 "" H 5150 900 60  0000 C CNN
-F 3 "" H 5150 900 60  0000 C CNN
-	1    5150 900
-	0    1    1    0
 $EndComp
 $Comp
@@
 $EndComp
 $Comp
-L GND #PWR040
+L GND #PWR047
 U 1 1 535DABD0
 P 5350 1700
-F 0 "#PWR040" H 5350 1700 30  0001 C CNN
+F 0 "#PWR047" H 5350 1700 30  0001 C CNN
 F 1 "GND" H 5350 1630 30  0001 C CNN
 F 2 "" H 5350 1700 60  0000 C CNN
@@
 Connection ~ 4850 1500
 Wire Wire Line
-	5350 900  5350 1700
-Wire Wire Line
 	4600 2300 4600 900
 Connection ~ 5350 1500
@@
 Connection ~ 4400 3600
 $Comp
-L GND #PWR041
+L GND #PWR048
 U 1 1 535DB671
 P 4400 4500
-F 0 "#PWR041" H 4400 4500 30  0001 C CNN
+F 0 "#PWR048" H 4400 4500 30  0001 C CNN
 F 1 "GND" H 4400 4430 30  0001 C CNN
 F 2 "" H 4400 4500 60  0000 C CNN
@@
 L R R10
 U 1 1 535DB823
-P 4600 2900
-F 0 "R10" V 4680 2900 40  0000 C CNN
-F 1 "10K" V 4607 2901 40  0000 C CNN
-F 2 "" V 4530 2900 30  0000 C CNN
-F 3 "" H 4600 2900 30  0000 C CNN
-	1    4600 2900
-	1    0    0    -1
-$EndComp
-$Comp
-L +5V #PWR042
+P 4300 2900
+F 0 "R10" V 4380 2900 40  0000 C CNN
+F 1 "10K" V 4307 2901 40  0000 C CNN
+F 2 "" V 4230 2900 30  0000 C CNN
+F 3 "" H 4300 2900 30  0000 C CNN
+	1    4300 2900
+	1    0    0    -1
+$EndComp
+$Comp
+L +5V #PWR049
 U 1 1 535DB86E
-P 4600 2550
-F 0 "#PWR042" H 4600 2640 20  0001 C CNN
-F 1 "+5V" H 4600 2640 30  0000 C CNN
-F 2 "" H 4600 2550 60  0000 C CNN
-F 3 "" H 4600 2550 60  0000 C CNN
-	1    4600 2550
-	1    0    0    -1
-$EndComp
-Wire Wire Line
-	4600 2550 4600 2650
+P 4450 2550
+F 0 "#PWR049" H 4450 2640 20  0001 C CNN
+F 1 "+5V" H 4450 2640 30  0000 C CNN
+F 2 "" H 4450 2550 60  0000 C CNN
+F 3 "" H 4450 2550 60  0000 C CNN
+	1    4450 2550
+	1    0    0    -1
+$EndComp
+Wire Wire Line
+	4450 2550 4450 2650
 Text HLabel 4050 2650 2    60   Input ~ 0
 A1
@@
 Text HLabel 4050 1700 2    60   BiDi ~ 0
 D8
-Connection ~ 4600 3150
+Connection ~ 4300 3150
 Wire Wire Line
 	3950 2650 4050 2650
@@
 $EndComp
 $Comp
-L GND #PWR043
+L GND #PWR050
 U 1 1 535E3E67
 P 6700 2800
-F 0 "#PWR043" H 6700 2800 30  0001 C CNN
+F 0 "#PWR050" H 6700 2800 30  0001 C CNN
 F 1 "GND" H 6700 2730 30  0001 C CNN
 F 2 "" H 6700 2800 60  0000 C CNN
@@
 	6100 2700 6200 2700
 Connection ~ 6100 2200
+Wire Wire Line
+	5350 900  5350 1700
+$Comp
+L Capacitor-General_EN60617-4_04-02-01_Date20121108 C6
+U 1 1 535DAAC1
+P 5150 900
+F 0 "C6" H 5200 1000 50  0000 L CNN
+F 1 "22pf" H 4950 1000 50  0000 L CNN
+F 2 "" H 5150 900 60  0000 C CNN
+F 3 "" H 5150 900 60  0000 C CNN
+	1    5150 900
+	0    1    1    0
+$EndComp
+$Comp
+L DIODE D8
+U 1 1 535FA04B
+P 4600 2850
+F 0 "D8" H 4600 2950 40  0000 C CNN
+F 1 "1N4001" H 4600 2750 40  0000 C CNN
+F 2 "" H 4600 2850 60  0000 C CNN
+F 3 "" H 4600 2850 60  0000 C CNN
+	1    4600 2850
+	0    -1   -1   0
+$EndComp
+Wire Wire Line
+	4600 3050 4600 3150
+Connection ~ 4600 3150
+Wire Wire Line
+	4300 2650 4600 2650
+Connection ~ 4450 2650
+$Comp
+L CRYSTAL X1
+U 1 1 535FCF6A
+P 4850 1200
+F 0 "X1" H 4850 1350 60  0000 C CNN
+F 1 "16.00MHz" H 4850 1050 60  0000 C CNN
+F 2 "" H 4850 1200 60  0000 C CNN
+F 3 "" H 4850 1200 60  0000 C CNN
+	1    4850 1200
+	0    1    1    0
+$EndComp
 $EndSCHEMATC
