File: KiCad/Mainboard/Floorboard.kicad_pcb (KiCad board)
At the start: 2 copper layers, 71 parts, among them IC1 ATMEGA328P-P, K1 CONN_3, K2 CONN_3, K3 CONN_3, K4 CONN_3, K5 CONN_3, K6 CONN_3, K7 CONN_3, K8 CONN_3, P1 CONN_4, P10 CONN_5, P11 CONN_5, P12 CONN_5, P13 CONN_5, P14 CONN_5, P15 CONN_6, P16 CONN_6, P17 CONN_5, P18 CONN_5, P19 CONN_5, P2 CONN_6, P20 CONN_5, P21 CONN_5, P22 CONN_6, P23 CONN_6, P24 CONN_3X2, P25 CONN_6, P26 CONN_2, P3 CONN_6, P4 CONN_6, P5 CONN_6, P6 CONN_6, P7 CONN_6, P8 CONN_6, P9 CONN_6, SW1 POWER_SEL, SW2 SW_PUSH, U1 LM7805CT, U2 MAX3100, U3 74LS138, U4 74LS138, U5 25LC1024, U6 4051, U7 74LS125, U8 74LS125, X1 16.00MHz, Y1 4MHz

Commit message: Initial Board Layout
Parts:
- added C10: 0.1uF, discret:C1, F.Cu at (199.4, 73.7)
- added C11: 0.1uF, discret:C1, F.Cu at (188.0, 78.7)
- added C12: 0.1uF, discret:C1, F.Cu at (188.0, 69.8)
- added C13: 0.1uF, discret:C1, F.Cu at (199.4, 78.7)
- added C14: 0.1uF, discret:C1, F.Cu at (198.1, 69.8)
- added C8: 0.1uF, discret:C1, F.Cu at (175.3, 73.7)
- added C9: 0.1uF, discret:C1, F.Cu at (188.0, 73.7)
- added D7: 1N4007, discret:D4, F.Cu at (31.8, 53.3)
- added D8: 1N4001, discret:D4, F.Cu at (66.0, 36.8)
- D2, D3: footprint led:LED-5MM -> led:LED-3MM
- K1, K2, K3, K4, K5, K6, K7, K8: footprint pin_array:PIN_ARRAY_3X1 -> TE_Connectivity:TE_CONN_EI_3
- P1: footprint pin_array:PIN_ARRAY_4x1 -> TE_Connectivity:TE_CONN_EI_4
- P10, P11, P12, P13, P14, P17, P18, P19, P20, P21: footprint pin_array:PIN_ARRAY_5x1 -> TE_Connectivity:TE_CONN_EI_5
- P15, P16, P2, P22, P23, P3, P4, P5, P6, P7, P8, P9: footprint pin_array:PIN_ARRAY-6X1 -> TE_Connectivity:TE_CONN_EI_6
- P26: footprint connect:SIL-2 -> TE_Connectivity:TE_CONN_TERM_2
- R2: value R -> 4.7K
- U1: footprint discret:TO220_VERT -> powerint:TO-220
- moved P1 103.7 mm to (141.0, 139.7)
- moved U2 103.7 mm to (144.8, 148.6)
- moved U8 103.3 mm to (190.5, 33.0)
- moved U7 101.5 mm to (190.5, 47.0)
- moved C5 80.2 mm to (54.6, 31.8), turned to 180 degrees
- moved C7 68.3 mm to (88.9, 27.9), turned to 90 degrees
- moved K8 68.1 mm to (273.1, 163.8)
- moved K5 68.1 mm to (273.1, 148.6)
- moved K4 67.9 mm to (273.1, 143.5)
- moved K7 67.9 mm to (273.1, 158.8)
- moved K3 67.7 mm to (273.1, 138.4)
- moved K6 67.7 mm to (273.1, 153.7)
- moved K2 67.6 mm to (273.1, 133.3)
- moved K1 67.5 mm to (273.1, 128.3)
- moved U6 67.4 mm to (246.4, 130.8)
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Other:
- board text added: "INPUT HEADERS"
- board text added: "OUTPUT HEADERS"
