File: KiCad/Mainboard/Floorboard.sch (KiCad schematic (older format))
At the start: 13 parts, among them P26 CONN_2, SW1 POWER_SEL, U1 LM7805CT

Commit message: Initial Board Layout
Parts:
- added D7: 1N4007, symbol DIODE
Connections:
- net +9V: now also D7.2 (K)
- net at C3.1, C4.1, SW1.1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: now also D7.1 (A)
Other:
- moved on the sheet: C1, C2, C3, C4, D1, D2, D4, D5, D6, P26, R1, SW1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
