File: KiCad/Mainboard/IO_Board.sch (KiCad schematic (older format))
At the start: 47 parts, among them K1 CONN_3, K2 CONN_3, K3 CONN_3, K4 CONN_3, K5 CONN_3, K6 CONN_3, K7 CONN_3, K8 CONN_3, P1 CONN_4, P10 CONN_5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

Commit message: Initial Board Layout
Parts:
- added C10, C11, C12, C13, C14, C8, C9: 0.1uF, symbol Capacitor-Mini
- R2: value R -> 4.7K
Connections:
- net +5V: now also C10.1, C11.1, C12.1, C13.2, C14.2, C8.1, C9.1
- net GND: now also C10.2, C11.2, C12.2, C13.1, C14.1, C8.2, C9.2
Other:
- moved on the sheet: U3
